Commit message: add table_circle

File: furniture_table_circle/table.urdf (robot description, URDF)
Before this commit: robot cube, 1 links, 0 joints
Links:
- link baseLink: mass 1.0 -> 15.0; geometry collision mesh filename=table.obj scale=0.02 0.02 0.02; visual mesh filename=table.obj scale=0.02 0.02 0.02
