Commit message: remove ply

File: utensil_knife_blue/model.urdf (robot description, URDF)
Before this commit: robot model.urdf, 1 links, 0 joints
Links:
- link baseLink: geometry collision mesh filename=collision.obj scale=0.8 0.8 0.8; visual mesh filename=textured.obj scale=0.8 0.8 0.8

File: utensil_plate_circle_green_big/model.urdf (robot description, URDF)
Before this commit: robot model.urdf, 1 links, 0 joints
Links:
- link baseLink: geometry collision mesh filename=collision.obj scale=1.2 1.2 1.2; visual mesh filename=textured.obj scale=1.2 1.2 1.2
