Commit message: update

File: utensil_mat_blue/model.urdf (robot description, URDF)
Before this commit: robot model.urdf, 1 links, 0 joints
Links:
- link baseLink: geometry collision mesh filename=textured.obj scale=1 1 1; visual mesh filename=textured.obj scale=1 1 1

Commit message: update

File: utensil_mat_blue/model.urdf (robot description, URDF)
Before this commit: robot model.urdf, 1 links, 0 joints
Links:
- link baseLink: geometry collision mesh filename=textured.dae scale=1 1 1; visual mesh filename=textured.dae scale=1 1 1

File: utensil_mat_blue_big/model.urdf (robot description, URDF)
Before this commit: robot model.urdf, 1 links, 0 joints
Links:
- link baseLink: geometry collision mesh filename=textured.dae scale=1.2 1.2 1.2; visual mesh filename=textured.dae scale=1.2 1.2 1.2

File: utensil_mat_blue_small/model.urdf (robot description, URDF)
Before this commit: robot model.urdf, 1 links, 0 joints
Links:
- link baseLink: geometry collision mesh filename=textured.dae scale=0.8 0.8 0.8; visual mesh filename=textured.dae scale=0.8 0.8 0.8

File: utensil_mat_green/model.urdf (robot description, URDF)
Before this commit: robot model.urdf, 1 links, 0 joints
Links:
- link baseLink: geometry collision mesh filename=textured.dae scale=1 1 1; visual mesh filename=textured.dae scale=1 1 1

File: utensil_mat_green_big/model.urdf (robot description, URDF)
Before this commit: robot model.urdf, 1 links, 0 joints
Links:
- link baseLink: geometry collision mesh filename=textured.dae scale=1.2 1.2 1.2; visual mesh filename=textured.dae scale=1.2 1.2 1.2

File: utensil_mat_green_small/model.urdf (robot description, URDF)
Before this commit: robot model.urdf, 1 links, 0 joints
Links:
- link baseLink: geometry collision mesh filename=textured.dae scale=0.8 0.8 0.8; visual mesh filename=textured.dae scale=0.8 0.8 0.8

File: utensil_mat_red/model.urdf (robot description, URDF)
Before this commit: robot model.urdf, 1 links, 0 joints
Links:
- link baseLink: geometry collision mesh filename=textured.dae scale=1.0 1.0 1.0; visual mesh filename=textured.dae scale=1.0 1.0 1.0

File: utensil_mat_red_big/model.urdf (robot description, URDF)
Before this commit: robot model.urdf, 1 links, 0 joints
Links:
- link baseLink: geometry collision mesh filename=textured.dae scale=1.2 1.2 1.2; visual mesh filename=textured.dae scale=1.2 1.2 1.2

File: utensil_mat_red_small/model.urdf (robot description, URDF)
Before this commit: robot model.urdf, 1 links, 0 joints
Links:
- link baseLink: geometry collision mesh filename=textured.dae scale=0.8 0.8 0.8; visual mesh filename=textured.dae scale=0.8 0.8 0.8
