Commit message: size

File: utensil_bowl_blue_small/model.urdf (robot description, URDF)
Before this commit: robot model.urdf, 1 links, 0 joints
Links:
- link baseLink: geometry collision mesh filename=collision.obj scale=0.85 0.85 0.85; visual mesh filename=textured.obj scale=0.85 0.85 0.85

File: utensil_fork_blue/model.urdf (robot description, URDF)
Before this commit: robot model.urdf, 1 links, 0 joints
Links:
- link baseLink: geometry collision mesh filename=collision.obj scale=1 1 1; visual mesh filename=textured.obj scale=1 1 1

File: utensil_napkin/model.urdf (robot description, URDF)
Before this commit: robot model.urdf, 1 links, 0 joints
Links:
- link baseLink: geometry collision mesh filename=texture.obj scale=1 1 1; visual mesh filename=texture.obj scale=1 1 1
