Commit message: update

File: utensil_napkin_blue/model.urdf (robot description, URDF)
Before this commit: robot model.urdf, 1 links, 0 joints
Links:
- link baseLink: geometry collision mesh filename=textured.dae scale=1 1 1; visual mesh filename=textured.dae scale=1 1 1

File: utensil_napkin_red/model.urdf (robot description, URDF)
Before this commit: robot model.urdf, 1 links, 0 joints
Links:
- link baseLink: geometry collision mesh filename=textured.dae scale=1 1 1; visual mesh filename=textured.dae scale=1 1 1
