Commit message: update

File: utensil_cup_blue/model.urdf (robot description, URDF)
Before this commit: robot model.urdf, 1 links, 0 joints
Links:
- link baseLink: geometry collision mesh filename=textured.dae scale=1 1 1; visual mesh filename=textured.dae scale=1 1 1

File: utensil_cup_blue_big/model.urdf (robot description, URDF)
Before this commit: robot model.urdf, 1 links, 0 joints
Links:
- link baseLink: geometry collision mesh filename=textured.dae scale=1.2 1.2 1.2; visual mesh filename=textured.dae scale=1.2 1.2 1.2

File: utensil_cup_blue_small/model.urdf (robot description, URDF)
Before this commit: robot model.urdf, 1 links, 0 joints
Links:
- link baseLink: geometry collision mesh filename=textured.dae scale=0.85 0.85 0.85; visual mesh filename=textured.dae scale=0.85 0.85 0.85

File: utensil_cup_green/model.urdf (robot description, URDF)
Before this commit: robot model.urdf, 1 links, 0 joints
Links:
- link baseLink: geometry collision mesh filename=textured.dae scale=1 1 1; visual mesh filename=textured.dae scale=1 1 1

File: utensil_cup_green_big/model.urdf (robot description, URDF)
Before this commit: robot model.urdf, 1 links, 0 joints
Links:
- link baseLink: geometry collision mesh filename=textured.dae scale=1.2 1.2 1.2; visual mesh filename=textured.dae scale=1.2 1.2 1.2

File: utensil_cup_green_small/model.urdf (robot description, URDF)
Before this commit: robot model.urdf, 1 links, 0 joints
Links:
- link baseLink: geometry collision mesh filename=textured.dae scale=0.85 0.85 0.85; visual mesh filename=textured.dae scale=0.85 0.85 0.85

File: utensil_cup_red/model.urdf (robot description, URDF)
Before this commit: robot model.urdf, 1 links, 0 joints
Links:
- link baseLink: geometry collision mesh filename=textured.dae scale=1 1 1; visual mesh filename=textured.dae scale=1 1 1

File: utensil_cup_red_big/model.urdf (robot description, URDF)
Before this commit: robot model.urdf, 1 links, 0 joints
Links:
- link baseLink: geometry collision mesh filename=textured.dae scale=1.2 1.2 1.2; visual mesh filename=textured.dae scale=1.2 1.2 1.2

File: utensil_cup_red_small/model.urdf (robot description, URDF)
Before this commit: robot model.urdf, 1 links, 0 joints
Links:
- link baseLink: geometry collision mesh filename=textured.dae scale=0.85 0.85 0.85; visual mesh filename=textured.dae scale=0.85 0.85 0.85
