Commit message: update

File: utensil_teacup_blue/model.urdf (robot description, URDF)
Before this commit: robot model.urdf, 1 links, 0 joints
Links:
- link baseLink: geometry collision mesh filename=collision.obj scale=1 1 1; visual mesh filename=textured.obj scale=1 1 1

File: utensil_teacup_blue_big/model.urdf (robot description, URDF)
Before this commit: robot model.urdf, 1 links, 0 joints
Links:
- link baseLink: geometry collision mesh filename=collision.obj scale=1.2 1.2 1.2; visual mesh filename=textured.obj scale=1.2 1.2 1.2

File: utensil_teacup_green/model.urdf (robot description, URDF)
Before this commit: robot model.urdf, 1 links, 0 joints
Links:
- link baseLink: geometry collision mesh filename=collision.obj scale=1 1 1; visual mesh filename=textured.obj scale=1 1 1

File: utensil_teacup_green_big/model.urdf (robot description, URDF)
Before this commit: robot model.urdf, 1 links, 0 joints
Links:
- link baseLink: geometry collision mesh filename=collision.obj scale=1.2 1.2 1.2; visual mesh filename=textured.obj scale=1.2 1.2 1.2

File: utensil_teacup_red/model.urdf (robot description, URDF)
Before this commit: robot model.urdf, 1 links, 0 joints
Links:
- link baseLink: geometry collision mesh filename=collision.obj scale=1 1 1; visual mesh filename=textured.obj scale=1 1 1

File: utensil_teacup_red_big/model.urdf (robot description, URDF)
Before this commit: robot model.urdf, 1 links, 0 joints
Links:
- link baseLink: geometry collision mesh filename=collision.obj scale=1.2 1.2 1.2; visual mesh filename=textured.obj scale=1.2 1.2 1.2
