Commit message: update

File: furniture_table_rectangle_high/table.urdf (robot description, URDF)
Before this commit: robot table.urdf, 1 links, 0 joints
Links:
- added link leg1; collision box size=0.1 0.1 0.95; visual mesh filename=table.obj scale=0.1 0.1 0.95
- added link leg2; collision box size=0.1 0.1 0.95; visual mesh filename=table.obj scale=0.1 0.1 0.95
- added link leg3; collision box size=0.1 0.1 0.95; visual mesh filename=table.obj scale=0.1 0.1 0.95
- added link leg4; collision box size=0.1 0.1 0.95; visual mesh filename=table.obj scale=0.1 0.1 0.95
- link baseLink: geometry collision box size=1.5 1 0.05; visual mesh filename=table.obj scale=1.5 1 0.05
Joints:
- added joint leg1_joint: type fixed, parent baseLink, child leg1
- added joint leg2_joint: type fixed, parent baseLink, child leg2
- added joint leg3_joint: type fixed, parent baseLink, child leg3
- added joint leg4_joint: type fixed, parent baseLink, child leg4
