Commit message: update

File: furniture_table_rectangle/table.urdf (robot description, URDF)
Before this commit: robot table.urdf, 1 links, 0 joints
Links:
- removed link baseLink
- added link leg1; collision cylinder length=0.7 radius=0.05; visual cylinder length=0.7 radius=0.05
- added link leg2; collision cylinder length=0.7 radius=0.05; visual cylinder length=0.7 radius=0.05
- added link leg3; collision cylinder length=0.7 radius=0.05; visual cylinder length=0.7 radius=0.05
- added link leg4; collision cylinder length=0.7 radius=0.05; visual cylinder length=0.7 radius=0.05
- added link table_top; collision box size=1.5 1 0.05; visual box size=1.5 1 0.05
Joints:
- added joint joint1: type fixed, parent table_top, child leg1, origin xyz=-0.65 -0.45 0 rpy=0 0 0
- added joint joint2: type fixed, parent table_top, child leg2, origin xyz=-0.65 0.45 0 rpy=0 0 0
- added joint joint3: type fixed, parent table_top, child leg3, origin xyz=0.65 -0.45 0 rpy=0 0 0
- added joint joint4: type fixed, parent table_top, child leg4, origin xyz=0.65 0.45 0 rpy=0 0 0
