Commit message: 更新 model.urdf 文件和添加新的 textured 文件

File: furniture_chair/model.urdf (robot description, URDF)
Before this commit: robot model.urdf, 1 links, 0 joints
Links:
- link baseLink: geometry collision mesh filename=textured.obj scale=0.85 0.85 0.85; visual mesh filename=textured.obj scale=0.85 0.85 0.85
